File: Cart_FeRAM/Cart_FeRAM.sch (KiCad schematic (older format))
At the start: 14 parts, among them CON1 GENESIS-EDGE, J1 Conn_01x32_Male, J2 Conn_01x32_Male, SW1 SW_DIP_x04, U1 74HC74, U2 FM1808B-SG, U3 74LS139, U4 27C322

Commit message: Updated board design, some project clean up
Parts:
- added JP1: <2M/4M, Jumper:SolderJumper-3_P1.3mm_Open_Pad1.0x1.5mm, symbol Jumper:Jumper_3_Open
- added R1, R2, R3, R4: 1K, Resistor_THT:R_Axial_DIN0207_L6.3mm_D2.5mm_P7.62mm_Horizontal, symbol Device:R
Connections:
- net labels added: CART_A17, CART_A18, CART_A19, CART_A20
- wire segments 81 -> 89
Other:
- moved on the sheet: SW1, U1B, U1C, U3A, U3B
